File: Si4825_KIT_TH.sch (EAGLE design)
At the start: 26 parts, among them U1 SI4825, U2 LMV358SOIC, Y1 32.768kHz

Commit message: Fixed issues discovered in first build
- fixed potentiometer footprint
- bigger strain relief holes: .1” to .15”
- changed U2 (op amp) to through hole version
- changed value of C9 (AC coupling capacitor) to 22uF in BOM and
schematic
- Removed R8 (jumper to bypass op amp)
- Regenerated gerbers, jpg previews, and pdf of schematic
Parts:
- removed R8: 0, SparkFun-Resistors:RESISTORAXIAL-0.3
- C9: value 1uF -> 22uF
- U2: value LMV358SOIC -> LM358; device SparkFun-AnalogIC:LMV358SOIC -> SparkFun-AnalogIC:LM358
Connections:
- net GND: now also U2G1.V-; no longer U2G1.GND
- net N$13: now also U2G1.-IN, U2G1.OUT; no longer R8.2, U2G1.-IN1, U2G1.OUT1
- net N$14: now also U2G1.+IN; no longer R8.1, U2G1.+IN1
- net V+: no longer U2G1.+V
Other:
- note added: "MCP6002-E/P"
- note removed: "MCP6002T-I/SN"
- note removed: "Stuff EITHER R8 or U2"
Changed lines of the file:
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@@
 <part name="C2" library="SparkFun-Capacitors" deviceset="CAP" device="PTH2" value="22pF"/>
 <part name="D1" library="SparkFun-DiscreteSemi" deviceset="DIODE" device="PTH"/>
-<part name="U2" library="SparkFun-AnalogIC" deviceset="LMV358" device="SOIC"/>
 <part name="SUPPLY17" library="supply2" deviceset="GND" device=""/>
 <part name="SUPPLY19" library="supply2" deviceset="V+" device=""/>
 <part name="C8" library="SparkFun-Capacitors" deviceset="CAP" device="_" value="1uF"/>
-<part name="C9" library="SparkFun-Capacitors" deviceset="CAP" device="_" value="1uF"/>
-<part name="R8" library="SparkFun-Resistors" deviceset="RESISTOR" device="AXIAL-0.3" value="0"/>
+<part name="C9" library="SparkFun-Capacitors" deviceset="CAP" device="_" value="22uF"/>
+<part name="U2" library="SparkFun-AnalogIC" deviceset="LM358" device=""/>
 </parts>
 <sheets>
@@
 <text x="22.86" y="35.56" size="1.778" layer="91">ANTENNA</text>
 <text x="66.04" y="60.96" size="1.778" layer="91">Si4825</text>
-<text x="86.36" y="91.44" size="1.778" layer="91">MCP6002T-I/SN</text>
-<text x="104.14" y="101.6" size="1.778" layer="91">Stuff EITHER R8 or U2</text>
+<text x="86.36" y="91.44" size="1.778" layer="91">MCP6002-E/P</text>
 </plain>
 <instances>
@@
 <attribute name="VALUE" x="30.2514" y="93.98" size="1.778" layer="96" rot="R90"/>
 </instance>
-<instance part="U2" gate="G1" x="116.84" y="76.2" smashed="yes">
-<attribute name="NAME" x="121.92" y="78.74" size="1.778" layer="95"/>
-</instance>
-<instance part="U2" gate="G2" x="144.78" y="50.8"/>
-<instance part="SUPPLY17" gate="GND" x="116.84" y="66.04"/>
-<instance part="SUPPLY19" gate="1" x="116.84" y="86.36"/>
+<instance part="SUPPLY17" gate="GND" x="114.3" y="63.5"/>
+<instance part="SUPPLY19" gate="1" x="114.3" y="88.9"/>
 <instance part="C8" gate="G$1" x="15.24" y="91.44"/>
 <instance part="C9" gate="G$1" x="139.7" y="76.2" smashed="yes" rot="R90">
@@
 <attribute name="VALUE" x="136.779" y="71.374" size="1.778" layer="96"/>
 </instance>
-<instance part="R8" gate="G$1" x="101.6" y="83.82"/>
+<instance part="U2" gate="G1" x="114.3" y="76.2"/>
 </instances>
 <busses>
@@
 </segment>
 <segment>
-<pinref part="U2" gate="G1" pin="+V"/>
 <pinref part="SUPPLY19" gate="1" pin="V+"/>
-<wire x1="116.84" y1="81.28" x2="116.84" y2="83.82" width="0.1524" layer="91"/>
+<wire x1="114.3" y1="83.82" x2="114.3" y2="86.36" width="0.1524" layer="91"/>
 </segment>
 </net>
@@
 </segment>
 <segment>
+<pinref part="U2" gate="G1" pin="V-"/>
 <pinref part="SUPPLY17" gate="GND" pin="GND"/>
-<pinref part="U2" gate="G1" pin="GND"/>
-<wire x1="116.84" y1="68.58" x2="116.84" y2="71.12" width="0.1524" layer="91"/>
+<wire x1="114.3" y1="66.04" x2="114.3" y2="68.58" width="0.1524" layer="91"/>
 </segment>
 </net>
@@
 <net name="N$13" class="0">
 <segment>
-<pinref part="U2" gate="G1" pin="OUT1"/>
 <wire x1="124.46" y1="93.98" x2="124.46" y2="76.2" width="0.1524" layer="91"/>
 <pinref part="C9" gate="G$1" pin="1"/>
 <wire x1="134.62" y1="76.2" x2="124.46" y2="76.2" width="0.1524" layer="91"/>
+<wire x1="109.22" y1="93.98" x2="109.22" y2="78.74" width="0.1524" layer="91"/>
+<wire x1="124.46" y1="93.98" x2="109.22" y2="93.98" width="0.1524" layer="91"/>
+<pinref part="U2" gate="G1" pin="-IN"/>
+<pinref part="U2" gate="G1" pin="OUT"/>
 <junction x="124.46" y="76.2"/>
-<pinref part="U2" gate="G1" pin="-IN1"/>
-<wire x1="109.22" y1="93.98" x2="109.22" y2="83.82" width="0.1524" layer="91"/>
-<wire x1="109.22" y1="83.82" x2="109.22" y2="78.74" width="0.1524" layer="91"/>
-<wire x1="124.46" y1="93.98" x2="109.22" y2="93.98" width="0.1524" layer="91"/>
-<pinref part="R8" gate="G$1" pin="2"/>
-<wire x1="106.68" y1="83.82" x2="109.22" y2="83.82" width="0.1524" layer="91"/>
-<junction x="109.22" y="83.82"/>
 </segment>
 </net>
@@
 <pinref part="U1" gate="G$1" pin="AOUT"/>
 <wire x1="86.36" y1="55.88" x2="83.82" y2="55.88" width="0.1524" layer="91"/>
-<wire x1="86.36" y1="78.74" x2="93.98" y2="78.74" width="0.1524" layer="91"/>
-<wire x1="93.98" y1="78.74" x2="99.06" y2="78.74" width="0.1524" layer="91"/>
+<wire x1="86.36" y1="78.74" x2="99.06" y2="78.74" width="0.1524" layer="91"/>
 <wire x1="99.06" y1="78.74" x2="99.06" y2="73.66" width="0.1524" layer="91"/>
-<pinref part="U2" gate="G1" pin="+IN1"/>
 <wire x1="99.06" y1="73.66" x2="109.22" y2="73.66" width="0.1524" layer="91"/>
-<pinref part="R8" gate="G$1" pin="1"/>
-<wire x1="96.52" y1="83.82" x2="93.98" y2="83.82" width="0.1524" layer="91"/>
-<wire x1="93.98" y1="83.82" x2="93.98" y2="78.74" width="0.1524" layer="91"/>
-<junction x="93.98" y="78.74"/>
-</segment>
-</net>
+<pinref part="U2" gate="G1" pin="+IN"/>
+</segment>
+</net>
